File: Eagle/Board4/Board4.sch (EAGLE design)
At the start: 39 parts, among them IC1 ESP-WROOM-02FRONT-FACE

Commit message: 一旦没にしてましたが発売することになり復活 ・シルクを整理 ・EN端子やLEDの電流制限抵抗値を見直し
Parts:
- C1, C2, C3, C5: device resistor:C-EUC0603 -> resistor:C-EUC0805
- R1, R2, R4, R5, R6, R7: device _temp:R-EU_R0603 -> resistor:R-EU_R0603
- R10, R8, R9: value 2k2 -> 4k7; device _temp:R-EU_R0603 -> resistor:R-EU_R0603
Changed lines of the file:
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@@
 <part name="IC1" library="esp-wroom-02" deviceset="ESP-WROOM-02" device="FRONT-FACE" value="ESP-WROOM-02FRONT-FACE"/>
 <part name="+3V2" library="supply1" deviceset="+3V3" device=""/>
-<part name="R1" library="_temp" deviceset="R-EU_" device="R0603" value="4k7"/>
-<part name="R2" library="_temp" deviceset="R-EU_" device="R0603" value="4k7"/>
-<part name="R4" library="_temp" deviceset="R-EU_" device="R0603" value="4k7"/>
+<part name="R1" library="resistor" deviceset="R-EU_" device="R0603" value="4k7"/>
+<part name="R2" library="resistor" deviceset="R-EU_" device="R0603" value="4k7"/>
+<part name="R4" library="resistor" deviceset="R-EU_" device="R0603" value="4k7"/>
 <part name="SUPPLY1" library="supply2" deviceset="GND" device=""/>
 <part name="SUPPLY2" library="supply2" deviceset="GND" device=""/>
@@
 <part name="13" library="wirepad" deviceset="1,6/0,9" device=""/>
 <part name="4DA" library="wirepad" deviceset="1,6/0,9" device=""/>
-<part name="R5" library="_temp" deviceset="R-EU_" device="R0603" value="4k7"/>
-<part name="R6" library="_temp" deviceset="R-EU_" device="R0603" value="4k7"/>
+<part name="R5" library="resistor" deviceset="R-EU_" device="R0603" value="4k7"/>
+<part name="R6" library="resistor" deviceset="R-EU_" device="R0603" value="4k7"/>
 <part name="RX" library="wirepad" deviceset="1,6/0,9" device=""/>
 <part name="TX" library="wirepad" deviceset="1,6/0,9" device=""/>
@@
 <part name="16" library="wirepad" deviceset="1,6/0,9" device=""/>
 <part name="SJ2" library="SparkFun" deviceset="SOLDERJUMPER" device="NO" value="SCL/PU"/>
-<part name="R7" library="_temp" deviceset="R-EU_" device="R0603" value="4k7"/>
-<part name="C2" library="resistor" deviceset="C-EU" device="C0603" value="4.7u"/>
+<part name="R7" library="resistor" deviceset="R-EU_" device="R0603" value="4k7"/>
+<part name="C2" library="resistor" deviceset="C-EU" device="C0805" value="4.7u"/>
 <part name="GND" library="wirepad" deviceset="1,6/0,9" device=""/>
 <part name="SUPPLY3" library="supply2" deviceset="GND" device=""/>
@@
 <part name="+3V1" library="supply1" deviceset="+3V3" device=""/>
 <part name="SJ-IO13" library="SparkFun" deviceset="SOLDERJUMPER" device="NO"/>
-<part name="R8" library="_temp" deviceset="R-EU_" device="R0603" value="2k2"/>
+<part name="R8" library="resistor" deviceset="R-EU_" device="R0603" value="4k7"/>
 <part name="L13" library="adafruit" deviceset="LED" device="CHIP-LED0603" value="IO13"/>
-<part name="R9" library="_temp" deviceset="R-EU_" device="R0603" value="2k2"/>
+<part name="R9" library="resistor" deviceset="R-EU_" device="R0603" value="4k7"/>
 <part name="LED-RXD" library="adafruit" deviceset="LED" device="CHIP-LED0603" value="R"/>
-<part name="R10" library="_temp" deviceset="R-EU_" device="R0603" value="2k2"/>
+<part name="R10" library="resistor" deviceset="R-EU_" device="R0603" value="4k7"/>
 <part name="LED-TXD" library="adafruit" deviceset="LED" device="CHIP-LED0603" value="T"/>
 <part name="SUPPLY8" library="supply2" deviceset="GND" device=""/>
 <part name="WAKEUP" library="SparkFun" deviceset="SOLDERJUMPER" device="NO"/>
 <part name="15" library="wirepad" deviceset="1,6/0,9" device=""/>
-<part name="C1" library="resistor" deviceset="C-EU" device="C0603" value="10u"/>
-<part name="C3" library="resistor" deviceset="C-EU" device="C0603" value="10u"/>
-<part name="C5" library="resistor" deviceset="C-EU" device="C0603" value="10u"/>
+<part name="C1" library="resistor" deviceset="C-EU" device="C0805" value="10u"/>
+<part name="C3" library="resistor" deviceset="C-EU" device="C0805" value="10u"/>
+<part name="C5" library="resistor" deviceset="C-EU" device="C0805" value="10u"/>
 <part name="PG" library="wirepad" deviceset="1,6/0,9" device=""/>
 <part name="RST" library="wirepad" deviceset="1,6/0,9" device=""/>
