File: Eagle/Board1/Board1.brd (EAGLE design)
At the start: 50 x 28 mm, 44 parts, among them IC1 ESP-WROOM-02FRONT-FACE, IC2 NMJ2845-33

Commit message: ver 1.1 : EN直結, RESET/PROG端子追加 - ENのプルアップ抵抗をやめてVcc直結 - RESET/PROGのPADを追加
Parts:
- removed R3: 1k, _temp:R0603
- added IO0, RST': (no value), wirepad:1,6/0,8
Connections:
- removed net N$1: IC1.2, R3.1
- net +3V3: now also IC1.2; no longer R3.2
- net N$2: now also IO0.1
- net N$8: now also RST'.1
Routing:
- net N$7: track 25.8 -> 43.8 mm, vias 4 -> 3
- net N$1: track 16.8 -> 0.00 mm, vias 2 -> 0
- net N$10: track 56.2 -> 68.9 mm, vias 3 -> 1
- net N$2: track 31.4 -> 38.8 mm, vias 2 -> 0
- net N$14: track 57.5 -> 50.9 mm, vias 3 -> 4
- net N$8: track 67.8 -> 63.4 mm, vias 4 -> 2
- net N$13: track 62.0 -> 65.1 mm
- net GND: track 117.8 -> 119.6 mm, vias 7 -> 6
- net N$6: track 25.6 -> 24.2 mm, vias 3 -> 2
- net +3V3: track 84.5 -> 85.5 mm, vias 7 -> 5
- net N$11: track 24.9 -> 25.5 mm
- net N$5: track 25.1 -> 25.7 mm
Other:
- board text added: "ESP-WROOM-02 / Board1 ver 1.1 by TareObjects 2016-09-20"
- board text removed: "ESP-WROOM-02 / Board1 ver 1.0 by TareObjects 2016-02-29"
